File: KiCad/Monitor/Monitor.kicad_pcb (KiCad board)
At the start: 2 copper layers, 4 parts, among them J1 BMP280, J2 CCS811, U1 WeMos_D1_mini

Commit message: first design
Parts:
- J1: footprint Connector_PinHeader_2.54mm:PinHeader_1x04_P2.54mm_Vertical -> Monitor:BMP280
- J2: footprint Connector_PinHeader_2.54mm:PinHeader_1x08_P2.54mm_Vertical -> Monitor:CCS811
- moved J1 90.0 mm to (90.2, 54.6), turned to 90 degrees
- moved J2 84.6 mm to (90.2, 73.7), turned to 180 degrees
- moved D1 77.0 mm to (121.0, 44.5), turned to 180 degrees
- moved U1 42.7 mm to (100.3, 57.1)
Connections:
- J1 pad 1: +5V -> +3V3
Other:
- board text added: "CO2 SENSOR"
- board text added: "V1.0"
- board text added: "Wiebe Beeftink Daniel Kievit"

Commit message: fixed pcb
Parts:
- moved J1 35.3 mm to (117.0, 77.5), turned to 270 degrees
- moved J2 29.7 mm to (117.0, 61.0), turned to 0 degrees
- moved U1 15.8 mm to (84.5, 57.5)
Connections:
- U1 pad 8: Net-(U1-Pad8) -> +3V3
Routing:
- net scl: track 0.00 -> 53.7 mm
- net +3V3: track 0.00 -> 49.5 mm
- net sda: track 0.00 -> 40.0 mm
- net +5V: track 0.00 -> 39.3 mm
- net din: track 0.00 -> 34.1 mm
- added copper zone on B.Cu, net GND
- added copper zone on F.Cu, net GND
Other:
- board text added: "JLCJLCJLCJLC"

Commit message: yes
Parts:
- moved D1 0.50 mm to (120.5, 44.5), turned to 270 degrees
Connections:
- D1 pad 1: GND -> +5V
- D1 pad 3: +5V -> GND
Routing:
- net din: track 34.1 -> 30.9 mm
- net +5V: track 39.3 -> 42.1 mm
Changed lines of the file:
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@@
-(kicad_pcb (version 20171130) (host pcbnew "(5.1.10)-1")
+(kicad_pcb (version 20171130) (host pcbnew "(5.1.9)-1")
   (general
     (thickness 1.6)
     (drawings 4)
-    (tracks 29)
+    (tracks 30)
     (zones 0)
     (modules 4)
@@
       (usegerberadvancedattributes true)
       (creategerberjobfile true)
-      (excludeedgelayer true)
+      (excludeedgelayer false)
       (linewidth 0.100000)
       (plotframeref false)
@@
   )
   (module LED_SMD:LED_WS2812B_PLCC4_5.0x5.0mm_P3.2mm (layer F.Cu)
-    (at 121 44.5 180)
+    (at 120.5 44.5 270)
     (descr https://cdn-shop.adafruit.com/datasheets/WS2812B.pdf)
     (tags "LED RGB NeoPixel")
     (attr smd)
-    (fp_text reference D1 (at 0.05 0.05) (layer F.SilkS) hide
-      (effects (font (size 1 1) (thickness 0.15)))
-    )
-    (fp_text value WS2812B (at 0 -3.5) (layer F.Fab) hide
+    (fp_text reference D1 (at 0.05 0.05 90) (layer F.SilkS) hide
+      (effects (font (size 1 1) (thickness 0.15)))
+    )
+    (fp_text value WS2812B (at 0 -3.5 90) (layer F.Fab) hide
       (effects (font (size 1 1) (thickness 0.15)))
     )
@@
     (fp_line (start 3.65 2.75) (end 3.65 1.6) (layer F.SilkS) (width 0.12))
     (fp_circle (center 0 0) (end 0 -2) (layer F.Fab) (width 0.1))
-    (fp_text user %R (at 0 0) (layer F.Fab)
+    (fp_text user %R (at 0 0 90) (layer F.Fab)
       (effects (font (size 0.8 0.8) (thickness 0.15)))
     )
-    (fp_text user 1 (at -4.15 -1.6) (layer F.SilkS) hide
-      (effects (font (size 1 1) (thickness 0.15)))
-    )
-    (pad 1 smd rect (at -2.45 -1.6 180) (size 1.5 1) (layers F.Cu F.Paste F.Mask)
+    (fp_text user 1 (at -4.15 -1.6 90) (layer F.SilkS) hide
+      (effects (font (size 1 1) (thickness 0.15)))
+    )
+    (pad 1 smd rect (at -2.45 -1.6 270) (size 1.5 1) (layers F.Cu F.Paste F.Mask)
+      (net 4 +5V))
+    (pad 2 smd rect (at -2.45 1.6 270) (size 1.5 1) (layers F.Cu F.Paste F.Mask)
+      (net 2 "Net-(D1-Pad2)"))
+    (pad 4 smd rect (at 2.45 -1.6 270) (size 1.5 1) (layers F.Cu F.Paste F.Mask)
+      (net 3 din))
+    (pad 3 smd rect (at 2.45 1.6 270) (size 1.5 1) (layers F.Cu F.Paste F.Mask)
       (net 1 GND))
-    (pad 2 smd rect (at -2.45 1.6 180) (size 1.5 1) (layers F.Cu F.Paste F.Mask)
-      (net 2 "Net-(D1-Pad2)"))
-    (pad 4 smd rect (at 2.45 -1.6 180) (size 1.5 1) (layers F.Cu F.Paste F.Mask)
-      (net 3 din))
-    (pad 3 smd rect (at 2.45 1.6 180) (size 1.5 1) (layers F.Cu F.Paste F.Mask)
-      (net 4 +5V))
     (model ${KISYS3DMOD}/LED_SMD.3dshapes/LED_WS2812B_PLCC4_5.0x5.0mm_P3.2mm.wrl
       (at (xyz 0 0 0))
@@
     (effects (font (size 2.5 2.5) (thickness 0.625)))
   )
-  (segment (start 118.55 66.113058) (end 113.063058 71.6) (width 0.25) (layer F.Cu) (net 3))
-  (segment (start 118.55 46.1) (end 118.55 66.113058) (width 0.25) (layer F.Cu) (net 3))
-  (segment (start 108.76 71.6) (end 107.36 70.2) (width 0.25) (layer F.Cu) (net 3))
-  (segment (start 113.063058 71.6) (end 108.76 71.6) (width 0.25) (layer F.Cu) (net 3))
-  (segment (start 111.1 50.35) (end 111.1 52.1) (width 0.25) (layer F.Cu) (net 4))
+  (segment (start 122.1 58.079002) (end 122.1 46.95) (width 0.25) (layer F.Cu) (net 3))
+  (segment (start 111.474003 68.704999) (end 122.1 58.079002) (width 0.25) (layer F.Cu) (net 3))
+  (segment (start 108.855001 68.704999) (end 111.474003 68.704999) (width 0.25) (layer F.Cu) (net 3))
+  (segment (start 107.36 70.2) (end 108.855001 68.704999) (width 0.25) (layer F.Cu) (net 3))
   (segment (start 111.1 52.1) (end 109.9 52.1) (width 0.25) (layer F.Cu) (net 4))
   (segment (start 109.9 52.1) (end 105.5 56.5) (width 0.25) (layer F.Cu) (net 4))
   (segment (start 105.5 73.42) (end 107.36 75.28) (width 0.25) (layer F.Cu) (net 4))
   (segment (start 105.5 56.5) (end 105.5 73.42) (width 0.25) (layer F.Cu) (net 4))
-  (segment (start 118.55 42.9) (end 111.1 50.35) (width 0.25) (layer F.Cu) (net 4))
+  (segment (start 111.3 52.1) (end 111.1 52.1) (width 0.25) (layer F.Cu) (net 4))
+  (segment (start 121.35 42.05) (end 111.3 52.1) (width 0.25) (layer F.Cu) (net 4))
+  (segment (start 122.1 42.05) (end 121.35 42.05) (width 0.25) (layer F.Cu) (net 4))
   (segment (start 105 76) (end 105 67.48) (width 0.25) (layer B.Cu) (net 5))
   (segment (start 106 77) (end 105 76) (width 0.25) (layer B.Cu) (net 5))
@@
   (segment (start 123.377389 79.122611) (end 123.377389 73.184671) (width 0.25) (layer F.Cu) (net 22))
   (segment (start 120.5 82) (end 123.377389 79.122611) (width 0.25) (layer F.Cu) (net 22))
+  (zone (net 0) (net_name "") (layer F.Cu) (hatch edge 0.508)
+    (connect_pads (clearance 0.508))
+    (min_thickness 0.254)
+    (keepout (tracks allowed) (vias allowed) (copperpour not_allowed))
+    (fill (arc_segments 32) (thermal_gap 0.508) (thermal_bridge_width 0.508))
+    (polygon
+      (pts
+        (xy 109 51) (xy 109 56) (xy 83 56) (xy 83 51) (xy 85 49)
+        (xy 107 49)
+      )
+    )
+  )
+  (zone (net 1) (net_name GND) (layer F.Cu) (hatch edge 0.508)
+    (connect_pads (clearance 0.508))
+    (min_thickness 0.254)
+    (fill yes (arc_segments 32) (thermal_gap 0.508) (thermal_bridge_width 0.508))
+    (polygon
+      (pts
+        (xy 126 85) (xy 82 85) (xy 82 40) (xy 126 40)
+      )
+    )
+  )
   (zone (net 1) (net_name GND) (layer B.Cu) (hatch edge 0.508)
     (connect_pads (clearance 0.508))
@@
     (polygon
       (pts
-        (xy 125.5 84.5) (xy 82 84.5) (xy 82 40.5) (xy 125.5 40.5)
+        (xy 126 85) (xy 82 85) (xy 82 40) (xy 126 40)
       )
     )
-  )
-  (zone (net 1) (net_name GND) (layer F.Cu) (hatch edge 0.508)
-    (connect_pads (clearance 0.508))
-    (min_thickness 0.254)
-    (fill yes (arc_segments 32) (thermal_gap 0.508) (thermal_bridge_width 0.508))
-    (polygon
-      (pts
-        (xy 125.5 84.5) (xy 82 84.5) (xy 82 40.5) (xy 125.5 40.5)
-      )
-    )

Commit message: v1.1
Connections:
- J2 pad 1: +5V -> +3V3
Routing:
- net +3V3: track 49.5 -> 72.0 mm
- net +5V: track 42.1 -> 51.9 mm
- net din: track 30.9 -> 36.0 mm
- net scl: track 53.7 -> 51.7 mm
Other:
- board outline added: 44 x 45 mm
- board text added: "V1.1"
- board text removed: "V1.0"
Changed lines of the file:
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@@
-(kicad_pcb (version 20171130) (host pcbnew "(5.1.9)-1")
+(kicad_pcb (version 20171130) (host pcbnew "(5.1.10)-1")
   (general
     (thickness 1.6)
-    (drawings 4)
-    (tracks 30)
+    (drawings 8)
+    (tracks 36)
     (zones 0)
     (modules 4)
@@
       (net 7 "Net-(J2-Pad8)"))
     (pad 1 thru_hole rect (at -5.9 -8.9) (size 1.7 1.7) (drill 1) (layers *.Cu *.Mask)
-      (net 4 +5V))
+      (net 22 +3V3))
   )
   (module Monitor:BMP280 (layer F.Cu)
@@
     )
   )
+  (gr_line (start 82 85) (end 82 40) (layer Edge.Cuts) (width 0.05))
+  (gr_line (start 126 85) (end 82 85) (layer Edge.Cuts) (width 0.05))
+  (gr_line (start 126 40) (end 126 85) (layer Edge.Cuts) (width 0.05))
+  (gr_line (start 82 40) (end 126 40) (layer Edge.Cuts) (width 0.05))
   (gr_text JLCJLCJLCJLC (at 96 65.25) (layer F.SilkS)
     (effects (font (size 1 1) (thickness 0.15)))
@@
     (effects (font (size 1.4 1.4) (thickness 0.2)))
   )
-  (gr_text V1.0 (at 112.78 43.23) (layer F.SilkS)
+  (gr_text V1.1 (at 112.78 43.23) (layer F.SilkS)
     (effects (font (size 1.5 1.5) (thickness 0.3)))
   )
@@
     (effects (font (size 2.5 2.5) (thickness 0.625)))
   )
-  (segment (start 122.1 58.079002) (end 122.1 46.95) (width 0.25) (layer F.Cu) (net 3))
-  (segment (start 111.474003 68.704999) (end 122.1 58.079002) (width 0.25) (layer F.Cu) (net 3))
-  (segment (start 108.855001 68.704999) (end 111.474003 68.704999) (width 0.25) (layer F.Cu) (net 3))
-  (segment (start 107.36 70.2) (end 108.855001 68.704999) (width 0.25) (layer F.Cu) (net 3))
-  (segment (start 111.1 52.1) (end 109.9 52.1) (width 0.25) (layer F.Cu) (net 4))
-  (segment (start 109.9 52.1) (end 105.5 56.5) (width 0.25) (layer F.Cu) (net 4))
-  (segment (start 105.5 73.42) (end 107.36 75.28) (width 0.25) (layer F.Cu) (net 4))
-  (segment (start 105.5 56.5) (end 105.5 73.42) (width 0.25) (layer F.Cu) (net 4))
-  (segment (start 111.3 52.1) (end 111.1 52.1) (width 0.25) (layer F.Cu) (net 4))
-  (segment (start 121.35 42.05) (end 111.3 52.1) (width 0.25) (layer F.Cu) (net 4))
-  (segment (start 122.1 42.05) (end 121.35 42.05) (width 0.25) (layer F.Cu) (net 4))
-  (segment (start 105 76) (end 105 67.48) (width 0.25) (layer B.Cu) (net 5))
-  (segment (start 106 77) (end 105 76) (width 0.25) (layer B.Cu) (net 5))
-  (segment (start 111.94206 77) (end 106 77) (width 0.25) (layer B.Cu) (net 5))
-  (segment (start 105 67.48) (end 107.36 65.12) (width 0.25) (layer B.Cu) (net 5))
-  (segment (start 115.757389 73.184671) (end 111.94206 77) (width 0.25) (layer B.Cu) (net 5))
-  (segment (start 115.757389 64.377389) (end 115.757389 73.184671) (width 0.25) (layer B.Cu) (net 5))
-  (segment (start 111.1 59.72) (end 115.757389 64.377389) (width 0.25) (layer B.Cu) (net 5))
-  (segment (start 118.297389 64.377389) (end 118.297389 73.184671) (width 0.25) (layer B.Cu) (net 6))
-  (segment (start 111.1 57.18) (end 118.297389 64.377389) (width 0.25) (layer B.Cu) (net 6))
-  (segment (start 107.36 62.58) (end 103 66.94) (width 0.25) (layer B.Cu) (net 6))
-  (segment (start 103 66.94) (end 103 77) (width 0.25) (layer B.Cu) (net 6))
-  (segment (start 103 77) (end 105 79) (width 0.25) (layer B.Cu) (net 6))
-  (segment (start 112.48206 79) (end 118.297389 73.184671) (width 0.25) (layer B.Cu) (net 6))
-  (segment (start 105 79) (end 112.48206 79) (width 0.25) (layer B.Cu) (net 6))
+  (segment (start 107.36 70.2) (end 107.9048 70.2) (width 0.25) (layer F.Cu) (net 3))
+  (segment (start 107.36 70.2) (end 107.7 70.2) (width 0.25) (layer F.Cu) (net 3))
+  (segment (start 107.36 70.2) (end 108.1 70.2) (width 0.25) (layer F.Cu) (net 3))
+  (segment (start 108.1 70.2) (end 109.2 69.1) (width 0.25) (layer F.Cu) (net 3))
+  (segment (start 109.2 69.1) (end 109.2 50.8) (width 0.25) (layer F.Cu) (net 3))
+  (segment (start 109.2 50.8) (end 110.4 49.6) (width 0.25) (layer F.Cu) (net 3))
+  (segment (start 119.45 49.6) (end 122.1 46.95) (width 0.25) (layer F.Cu) (net 3))
+  (segment (start 110.4 49.6) (end 119.45 49.6) (width 0.25) (layer F.Cu) (net 3))
+  (segment (start 107.36 75.28) (end 123.97 75.28) (width 0.25) (layer F.Cu) (net 4))
+  (segment (start 123.97 75.28) (end 125.5 73.75) (width 0.25) (layer F.Cu) (net 4))
+  (segment (start 125.5 45.45) (end 122.1 42.05) (width 0.25) (layer F.Cu) (net 4))
+  (segment (start 125.5 73.75) (end 125.5 45.45) (width 0.25) (layer F.Cu) (net 4))
+  (segment (start 115.757389 64.377389) (end 111.1 59.72) (width 0.25) (layer F.Cu) (net 5))
+  (segment (start 115.757389 73.184671) (end 115.757389 64.377389) (width 0.25) (layer F.Cu) (net 5))
+  (segment (start 107.36 65.12) (end 107.36 65.14) (width 0.25) (layer B.Cu) (net 5))
+  (segment (start 107.36 65.12) (end 105.5 66.98) (width 0.25) (layer B.Cu) (net 5))
+  (segment (start 105.5 66.98) (end 105.5 76) (width 0.25) (layer B.Cu) (net 5))
+  (segment (start 105.5 76) (end 107 77.5) (width 0.25) (layer B.Cu) (net 5))
+  (segment (start 111.44206 77.5) (end 115.757389 73.184671) (width 0.25) (layer B.Cu) (net 5))
+  (segment (start 107 77.5) (end 111.44206 77.5) (width 0.25) (layer B.Cu) (net 5))
+  (segment (start 118.297389 64.377389) (end 118.297389 73.184671) (width 0.25) (layer F.Cu) (net 6))
+  (segment (start 111.1 57.18) (end 118.297389 64.377389) (width 0.25) (layer F.Cu) (net 6))
+  (segment (start 107.36 62.58) (end 107.36 62.566) (width 0.25) (layer F.Cu) (net 6))
+  (segment (start 107.36 62.58) (end 104 65.94) (width 0.25) (layer B.Cu) (net 6))
+  (segment (start 104 65.94) (end 104 76.25) (width 0.25) (layer B.Cu) (net 6))
+  (segment (start 104 76.25) (end 106.5 78.75) (width 0.25) (layer B.Cu) (net 6))
+  (segment (start 112.73206 78.75) (end 118.297389 73.184671) (width 0.25) (layer B.Cu) (net 6))
+  (segment (start 106.5 78.75) (end 112.73206 78.75) (width 0.25) (layer B.Cu) (net 6))
+  (segment (start 111.3 52.1) (end 111.1 52.1) (width 0.25) (layer F.Cu) (net 22))
   (segment (start 84.5 75.28) (end 83.78 75.28) (width 0.25) (layer B.Cu) (net 22))
-  (segment (start 84.5 75.28) (end 91.22 82) (width 0.25) (layer F.Cu) (net 22))
-  (segment (start 91.22 82) (end 120.5 82) (width 0.25) (layer F.Cu) (net 22))
-  (segment (start 123.377389 79.122611) (end 123.377389 73.184671) (width 0.25) (layer F.Cu) (net 22))
-  (segment (start 120.5 82) (end 123.377389 79.122611) (width 0.25) (layer F.Cu) (net 22))
+  (segment (start 123.377389 64.377389) (end 111.1 52.1) (width 0.25) (layer F.Cu) (net 22))
+  (segment (start 123.377389 73.184671) (end 123.377389 64.377389) (width 0.25) (layer F.Cu) (net 22))
+  (segment (start 84.5 75.28) (end 84.5 77.5) (width 0.25) (layer B.Cu) (net 22))
+  (segment (start 84.5 77.5) (end 87 80) (width 0.25) (layer B.Cu) (net 22))
+  (segment (start 116.56206 80) (end 123.377389 73.184671) (width 0.25) (layer B.Cu) (net 22))
+  (segment (start 87 80) (end 116.56206 80) (width 0.25) (layer B.Cu) (net 22))
   (zone (net 0) (net_name "") (layer F.Cu) (hatch edge 0.508)
     (connect_pads (clearance 0.508))
