File: KiCad/Monitor/Monitor.sch (KiCad schematic (older format))
At the start: 4 parts, among them J1 BMP280, J2 CCS811, U1 WeMos_D1_mini

Commit message: first design
Parts:
- removed J1: BMP280, Connector_PinHeader_2.54mm:PinHeader_1x04_P2.54mm_Vertical, symbol Connector:Conn_01x04_Male
- added J1: BMP280, Monitor:BMP280, symbol Connector:Conn_01x06_Male
- J2: footprint Connector_PinHeader_2.54mm:PinHeader_1x08_P2.54mm_Vertical -> Monitor:CCS811
Connections:
- net GND: now also J1.2 (Pin_2)
- net scl: now also J1.3 (Pin_3)
- net sda: now also J1.4 (Pin_4)
- new net +3V3: J1.1 (Pin_1)
Changed lines of the file:
@@
 Text GLabel 2450 2600 2    50   Input ~ 0
-sda
-Text GLabel 2950 2400 2    50   Input ~ 0
 sda
 $Comp
@@
 din
 $Comp
-L power:GND #PWR0104
-U 1 1 60B3EC77
-P 2950 2200
-F 0 "#PWR0104" H 2950 1950 50  0001 C CNN
-F 1 "GND" V 2955 2072 50  0000 R CNN
-F 2 "" H 2950 2200 50  0001 C CNN
-F 3 "" H 2950 2200 50  0001 C CNN
-	1    2950 2200
-	0    -1   -1   0
-$EndComp
-Text GLabel 2950 2300 2    50   Input ~ 0
-scl
-$Comp
-L power:+5V #PWR0103
-U 1 1 60B19272
-P 2950 2100
-F 0 "#PWR0103" H 2950 1950 50  0001 C CNN
-F 1 "+5V" V 2965 2228 50  0000 L CNN
-F 2 "" H 2950 2100 50  0001 C CNN
-F 3 "" H 2950 2100 50  0001 C CNN
-	1    2950 2100
-	0    1    1    0
-$EndComp
-$Comp
 L power:+5V #PWR0105
 U 1 1 60B432E3
@@
 $EndComp
 $Comp
-L Connector:Conn_01x04_Male J1
-U 1 1 60B2400F
-P 2750 2200
-F 0 "J1" H 2858 2481 50  0000 C CNN
-F 1 "BMP280" H 2858 2390 50  0000 C CNN
-F 2 "Connector_PinHeader_2.54mm:PinHeader_1x04_P2.54mm_Vertical" H 2750 2200 50  0001 C CNN
-F 3 "~" H 2750 2200 50  0001 C CNN
-	1    2750 2200
-	1    0    0    -1
-$EndComp
-$Comp
 L Connector:Conn_01x08_Male J2
 U 1 1 60B25397
@@
 F 0 "J2" H 2858 3481 50  0000 C CNN
 F 1 "CCS811" H 2858 3390 50  0000 C CNN
-F 2 "Connector_PinHeader_2.54mm:PinHeader_1x08_P2.54mm_Vertical" H 2750 3000 50  0001 C CNN
+F 2 "Monitor:CCS811" H 2750 3000 50  0001 C CNN
 F 3 "~" H 2750 3000 50  0001 C CNN
 	1    2750 3000
 	1    0    0    -1
 $EndComp
+$Comp
+L Connector:Conn_01x06_Male J1
+U 1 1 60B1AB60
+P 2750 2100
+F 0 "J1" H 2858 2481 50  0000 C CNN
+F 1 "BMP280" H 2858 2390 50  0000 C CNN
+F 2 "Monitor:BMP280" H 2750 2100 50  0001 C CNN
+F 3 "~" H 2750 2100 50  0001 C CNN
+	1    2750 2100
+	1    0    0    -1
+$EndComp
+$Comp
+L power:+3.3V #PWR01
+U 1 1 60B1CACD
+P 2950 1900
+F 0 "#PWR01" H 2950 1750 50  0001 C CNN
+F 1 "+3.3V" V 2965 2028 50  0000 L CNN
+F 2 "" H 2950 1900 50  0001 C CNN
+F 3 "" H 2950 1900 50  0001 C CNN
+	1    2950 1900
+	0    1    1    0
+$EndComp
+$Comp
+L power:GND #PWR02
+U 1 1 60B1D47D
+P 2950 2000
+F 0 "#PWR02" H 2950 1750 50  0001 C CNN
+F 1 "GND" V 2955 1872 50  0000 R CNN
+F 2 "" H 2950 2000 50  0001 C CNN
+F 3 "" H 2950 2000 50  0001 C CNN
+	1    2950 2000
+	0    -1   -1   0
+$EndComp
+Text GLabel 2950 2100 2    50   Input ~ 0
+scl
+Text GLabel 2950 2200 2    50   Input ~ 0
+sda
 $EndSCHEMATC

Commit message: fixed pcb
Connections:
- net +3V3: now also U1.8 (3V3)
Changed lines of the file:
@@
 Text GLabel 2950 2200 2    50   Input ~ 0
 sda
+$Comp
+L power:+3.3V #PWR?
+U 1 1 60B22B77
+P 2150 2000
+F 0 "#PWR?" H 2150 1850 50  0001 C CNN
+F 1 "+3.3V" H 2165 2173 50  0000 C CNN
+F 2 "" H 2150 2000 50  0001 C CNN
+F 3 "" H 2150 2000 50  0001 C CNN
+	1    2150 2000
+	1    0    0    -1
+$EndComp
 $EndSCHEMATC

Commit message: yes
Connections:
- net +5V: now also D1.1 (VDD); no longer D1.3 (VSS)
- net GND: now also D1.3 (VSS); no longer D1.1 (VDD)
Changed lines of the file:
@@
 L power:GND #PWR0108
 U 1 1 60B4A589
-P 3150 3550
-F 0 "#PWR0108" H 3150 3300 50  0001 C CNN
-F 1 "GND" V 3155 3422 50  0000 R CNN
-F 2 "" H 3150 3550 50  0001 C CNN
-F 3 "" H 3150 3550 50  0001 C CNN
-	1    3150 3550
-	-1   0    0    1
+P 3150 4150
+F 0 "#PWR0108" H 3150 3900 50  0001 C CNN
+F 1 "GND" V 3155 4022 50  0000 R CNN
+F 2 "" H 3150 4150 50  0001 C CNN
+F 3 "" H 3150 4150 50  0001 C CNN
+	1    3150 4150
+	1    0    0    -1
 $EndComp
 $Comp
 L power:+5V #PWR0109
 U 1 1 60B4EE1B
-P 3150 4150
-F 0 "#PWR0109" H 3150 4000 50  0001 C CNN
-F 1 "+5V" H 3165 4323 50  0000 C CNN
-F 2 "" H 3150 4150 50  0001 C CNN
-F 3 "" H 3150 4150 50  0001 C CNN
-	1    3150 4150
-	-1   0    0    1
+P 3150 3550
+F 0 "#PWR0109" H 3150 3400 50  0001 C CNN
+F 1 "+5V" H 3165 3723 50  0000 C CNN
+F 2 "" H 3150 3550 50  0001 C CNN
+F 3 "" H 3150 3550 50  0001 C CNN
+	1    3150 3550
+	1    0    0    -1
 $EndComp
 Text GLabel 2850 3850 0    50   Input ~ 0

Commit message: v1.1
Connections:
- net +3V3: now also J2.1 (Pin_1)
- net +5V: no longer J2.1 (Pin_1)
Changed lines of the file:
@@
 din
-$Comp
-L power:+5V #PWR0105
-U 1 1 60B432E3
-P 2950 2700
-F 0 "#PWR0105" H 2950 2550 50  0001 C CNN
-F 1 "+5V" V 2965 2828 50  0000 L CNN
-F 2 "" H 2950 2700 50  0001 C CNN
-F 3 "" H 2950 2700 50  0001 C CNN
-	1    2950 2700
-	0    1    1    0
-$EndComp
 $Comp
 L Connector:Conn_01x08_Male J2
@@
 	1    0    0    -1
 $EndComp
+$Comp
+L power:+3.3V #PWR?
+U 1 1 60C1C40B
+P 2950 2700
+F 0 "#PWR?" H 2950 2550 50  0001 C CNN
+F 1 "+3.3V" V 2965 2828 50  0000 L CNN
+F 2 "" H 2950 2700 50  0001 C CNN
+F 3 "" H 2950 2700 50  0001 C CNN
+	1    2950 2700
+	0    1    1    0
+$EndComp
 $EndSCHEMATC
